Commit message: Major update

File: rp_robot_description/urdf/rp_robot.urdf (robot description, URDF)
Before this commit: robot rp_robot, 3 links, 2 joints
Links:
- added link EE, mass 1000; collision sphere radius=0.1; visual sphere radius=0.1
Joints:
- added joint J02: type fixed, parent L02, child EE, origin xyz=0.0 0.0 0.875 rpy=0.0 0.0 0.0
- joint J00: limit effort=10000 velocity=0.5 -> lower=-1.3090 upper=4.4506 effort=10000 velocity=0.5; type continuous -> revolute
