Commit message: Updated values

File: rr_robot_description/urdf/rr_robot.urdf (robot description, URDF)
Before this commit: robot rr_robot, 4 links, 3 joints
Joints:
- joint J02: origin xyz=0.27276731 0.1042208 0.08 rpy=0.0 0.0 0.0 -> xyz=0.27276731 0.1042208 0.08000 rpy=0.0 0.0 0.0

Commit message: Updated location of EE-frame, it is now in the origin of EE its CoG

File: rr_robot_description/urdf/rr_robot.urdf (robot description, URDF)
Before this commit: robot rr_robot, 4 links, 3 joints
Joints:
- joint J03: origin xyz=0.435 0.0 0.0 rpy=0.0 0.0 0.0 -> xyz=0.505184 0.0 0.0 rpy=0.0 0.0 0.0

Commit message: Corrected izz which was written in iyz, also the mass and inertia have reduced to match 2kg EE

File: rr_robot_description/urdf/rr_robot.urdf (robot description, URDF)
Before this commit: robot rr_robot, 4 links, 3 joints
Links:
- link EE: mass 10.000 -> 2.000
