Commit message: Moved some files around

File: robots/rp_robot_description/urdf/rp_robot.urdf (robot description, URDF)
Before this commit: robot rr_robot, 4 links, 3 joints
Links:
- link EE: mass 2.000 -> 1000; geometry collision sphere radius=0.1; visual sphere radius=0.1
- link L00: mass 294.264 -> 456.291; geometry collision mesh filename=package://tameshiwari/robots/rp_robot_description/meshes/Li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 scale=1 1 1; visual mesh filename=package://tameshiwari/robots/rp_robot_description/meshes/Li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 scale=1 1 1
- link L01: mass 4.000 -> 54.677; geometry collision mesh filename=package://tameshiwari/robots/rp_robot_description/meshes/Li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 scale=1 1 1; visual mesh filename=package://tameshiwari/robots/rp_robot_description/meshes/Li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 scale=1 1 1
- link L02: mass 4.000 -> 17.606; geometry collision mesh filename=package://tameshiwari/robots/rp_robot_description/meshes/Li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 scale=1 1 1; visual mesh filename=package://tameshiwari/robots/rp_robot_description/meshes/Li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 scale=1 1 1
Joints:
- removed joint J03
- added joint J00: type revolute, parent L00, child L01, origin xyz=0.0 0.0 2.0 rpy=0.0 1.5707 0.0, axis 0.0 0.0 1.0, limit lower=-1.3090 upper=4.4506 effort=10000 velocity=0.5
- joint J01: child L01 -> L02; limit lower=-1.6580627893946132 upper=3.4033920413889427 effort=10000 velocity=0.5 -> lower=-0.37 upper=0.37 effort=1000.0 velocity=0.5; origin xyz=0.0 0.0 1.2 rpy=0.0 1.5707 0.0 -> xyz=0.57 0.0 0.0 rpy=0.0 1.5707 0.0; parent L00 -> L01; type revolute -> prismatic
- joint J02: axis 0.0 0.0 1.0 -> (none); child L02 -> EE; limit lower=-0.3490658503988659 upper=2.530727415391778 effort=1000.0 velocity=0.5 -> (none); origin xyz=0.27276731 0.1042208 0.08000 rpy=0.0 0.0 0.0 -> xyz=0.0 0.0 0.875 rpy=0.0 0.0 0.0; parent L01 -> L02; type revolute -> fixed

File: robots/rr_robot_description/urdf/rr_robot.urdf (robot description, URDF)
Before this commit: robot rp_robot, 4 links, 3 joints
Links:
- link EE: mass 1000 -> 2.000; geometry collision mesh filename=package://tameshiwari/robots/rr_robot_description/meshes/RR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 scale=1 1 1; visual mesh filename=package://tameshiwari/robots/rr_robot_description/meshes/RR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 scale=1 1 1
- link L00: mass 456.291 -> 294.264; geometry collision mesh filename=package://tameshiwari/robots/rr_robot_description/meshes/RR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 scale=1 1 1; visual mesh filename=package://tameshiwari/robots/rr_robot_description/meshes/RR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 scale=1 1 1
- link L01: mass 54.677 -> 4.000; geometry collision mesh filename=package://tameshiwari/robots/rr_robot_description/meshes/RR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 scale=1 1 1; visual mesh filename=package://tameshiwari/robots/rr_robot_description/meshes/RR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 scale=1 1 1
- link L02: mass 17.606 -> 4.000; geometry collision mesh filename=package://tameshiwari/robots/rr_robot_description/meshes/RR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 scale=1 1 1; visual mesh filename=package://tameshiwari/robots/rr_robot_description/meshes/RR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 scale=1 1 1
Joints:
- removed joint J00
- added joint J03: type fixed, parent L02, child EE, origin xyz=0.505184 0.0 0.0 rpy=0.0 0.0 0.0
- joint J01: child L02 -> L01; limit lower=-0.37 upper=0.37 effort=1000.0 velocity=0.5 -> lower=-1.6580627893946132 upper=3.4033920413889427 effort=10000 velocity=0.5; origin xyz=0.57 0.0 0.0 rpy=0.0 1.5707 0.0 -> xyz=0.0 0.0 1.2 rpy=0.0 1.5707 0.0; parent L01 -> L00; type prismatic -> revolute
- joint J02: axis (none) -> 0.0 0.0 1.0; child EE -> L02; limit (none) -> lower=-0.3490658503988659 upper=2.530727415391778 effort=1000.0 velocity=0.5; origin xyz=0.0 0.0 0.875 rpy=0.0 0.0 0.0 -> xyz=0.27276731 0.1042208 0.08000 rpy=0.0 0.0 0.0; parent L02 -> L01; type fixed -> revolute
