Commit message: Functional Optimal Tameshiwari --> real life test confirmed

File: robots/centauro_robot_description/config/joint_limits.xacro (robot description, xacro)
@@ -30,12 +30,20 @@
 <xacro:property name="j_arm_6_upper" value="${[1.509, 1.5156]}"/>
 <xacro:property name="j_arm_7_upper" value="${[2.569, 2.5686]}"/>
-<xacro:property name="j_arm_1_velocity" value="${[3.86, 3.86 ]}"/>
+<!-- <xacro:property name="j_arm_1_velocity" value="${[3.86, 3.86 ]}"/>
 <xacro:property name="j_arm_2_velocity" value="${[3.86, 3.86 ]}"/>
 <xacro:property name="j_arm_3_velocity" value="${[6.06, 6.06 ]}"/>
 <xacro:property name="j_arm_4_velocity" value="${[6.06, 6.06 ]}"/>
 <xacro:property name="j_arm_5_velocity" value="${[11.72, 11.72 ]}"/>
+<xacro:property name="j_arm_5_velocity" value="${[11.72, 11.72 ]}"/>
 <xacro:property name="j_arm_6_velocity" value="${[11.72, 11.72 ]}"/>
-<xacro:property name="j_arm_7_velocity" value="${[20.35, 20.35 ]}"/>
-<xacro:property name="j_arm_1_torque" value="${[147.00, 147.00 ]}"/>
+<xacro:property name="j_arm_7_velocity" value="${[20.35, 20.35 ]}"/> -->
+<xacro:property name="j_arm_1_velocity" value="${[6.00 6.00 ]}"/>
+<xacro:property name="j_arm_2_velocity" value="${[6.00 6.00 ]}"/>
+<xacro:property name="j_arm_3_velocity" value="${[6.00 6.00 ]}"/>
+<xacro:property name="j_arm_4_velocity" value="${[6.00 6.00 ]}"/>
+<xacro:property name="j_arm_5_velocity" value="${[6.00 6.00 ]]}"/>
+<xacro:property name="j_arm_6_velocity" value="${[6.00 6.00 ]}"/>
+<xacro:property name="j_arm_7_velocity" value="${[6.00 6.00 ]}"/>
+<!-- <xacro:property name="j_arm_1_torque" value="${[147.00, 147.00 ]}"/>
 <xacro:property name="j_arm_2_torque" value="${[147.00, 147.00 ]}"/>
 <xacro:property name="j_arm_3_torque" value="${[147.00, 147.00 ]}"/>
@@ -43,5 +51,12 @@
 <xacro:property name="j_arm_5_torque" value="${[55.00, 55.00 ]}"/>
 <xacro:property name="j_arm_6_torque" value="${[55.00, 55.00 ]}"/>
-<xacro:property name="j_arm_7_torque" value="${[28.32, 28.32 ]}"/>
+<xacro:property name="j_arm_7_torque" value="${[28.32, 28.32 ]}"/> -->
+<xacro:property name="j_arm_1_torque" value="${[140.00, 140.00 ]}"/>
+<xacro:property name="j_arm_2_torque" value="${[140.00, 140.00 ]}"/>
+<xacro:property name="j_arm_3_torque" value="${[120.00, 120.00 ]}"/>
+<xacro:property name="j_arm_4_torque" value="${[120.00, 120.00 ]}"/>
+<xacro:property name="j_arm_5_torque" value="${[35.00, 35.00 ]}"/>
+<xacro:property name="j_arm_6_torque" value="${[35.00, 35.00 ]}"/>
+<xacro:property name="j_arm_7_torque" value="${[20.00, 20.00 ]}"/>
 <xacro:property name="motor_A_velocity" value="8.8"/>
 <xacro:property name="motor_B_velocity" value="8.1"/>
