Commit message: working on initialization of centauro scripts

File: robots/centauro_robot_description/config/centauro_srdf.xacro (robot description, xacro)
@@ -1,4 +1,46 @@
 <?xml version="1.0"?>
 <robot name="centauro">
+   <group name="joint_names">
+        <joint name="j_arm1_1" />
+        <joint name="j_arm1_2" />
+        <joint name="j_arm1_3" />
+        <joint name="j_arm1_4" />
+        <joint name="j_arm1_5"/>
+        <joint name="j_arm1_6" />
+        <joint name="j_arm1_7"/>
+        <joint name="j_arm2_1"/>
+        <joint name="j_arm2_2"/>
+        <joint name="j_arm2_3"/>
+        <joint name="j_arm2_4" />
+        <joint name="j_arm2_5"/>
+        <joint name="j_arm2_6"/>
+        <joint name="j_arm2_7"/>
+        <joint name="hip_yaw_1"/>
+        <joint name="hip_pitch_1" />
+        <joint name="knee_pitch_1" />
+        <joint name="ankle_yaw_1"/>
+        <joint name="ankle_pitch_1"/>
+        <joint name="j_wheel_1" />
+        <joint name="hip_yaw_2"/>
+        <joint name="hip_pitch_2"/>
+        <joint name="knee_pitch_2"/>
+        <joint name="ankle_yaw_2" />
+        <joint name="ankle_pitch_2"/>
+        <joint name="j_wheel_2" />
+        <joint name="hip_yaw_3"/>
+        <joint name="hip_pitch_3"/>
+        <joint name="knee_pitch_3"/>
+        <joint name="ankle_yaw_3"/>
+        <joint name="ankle_pitch_3" />
+        <joint name="j_wheel_3" />
+        <joint name="hip_yaw_4"/>
+        <joint name="hip_pitch_4" />
+        <joint name="knee_pitch_4" />
+        <joint name="ankle_yaw_4" />
+        <joint name="ankle_pitch_4"/>
+        <joint name="j_wheel_4" />
+        <joint name="torso_yaw"/>
+        <joint name="neck_pitch" />
+   </group>
    <group name="velodyne">
       <chain base_link="torso_2" tip_link="neck_3"/>
@@ -65,8 +107,6 @@
    </group>
    <group_state name="home" group="chains">
-        <joint name="torso_yaw" value="0.0"/>
-        <joint name="neck_pitch" value="0.45"/>
         <joint name="j_arm1_1" value="0.5"/>
-        <joint name="j_arm1_2" value="-0.3"/>
+        <joint name="j_arm1_2" value="0.03"/>
         <joint name="j_arm1_3" value="-0.3"/>
         <joint name="j_arm1_4" value="-2.2"/>
@@ -74,8 +114,8 @@
         <joint name="j_arm1_6" value="-0.8"/>
         <joint name="j_arm1_7" value="0.0"/>
-        <joint name="j_arm2_1" value="-0.5"/>
-        <joint name="j_arm2_2" value="0.3"/>
+        <joint name="j_arm2_1" value="0.5"/>
+        <joint name="j_arm2_2" value="-0.03"/>
         <joint name="j_arm2_3" value="0.3"/>
-        <joint name="j_arm2_4" value="2.2"/>
+        <joint name="j_arm2_4" value="-2.2"/>
         <joint name="j_arm2_5" value="0.0"/>
         <joint name="j_arm2_6" value="0.8"/>
@@ -85,16 +125,26 @@
         <joint name="knee_pitch_1" value="-1.0"/>
         <joint name="ankle_yaw_1" value="-0.78"/>
+        <joint name="ankle_pitch_1" value="0.0"/>
+        <joint name="j_wheel_1" value="0.0" />
         <joint name="hip_yaw_2" value="0.0"/>
         <joint name="hip_pitch_2" value="1.0"/>
         <joint name="knee_pitch_2" value="1.0"/>
         <joint name="ankle_yaw_2" value="0.78"/>
+        <joint name="ankle_pitch_2" value="0.0"/>
+        <joint name="j_wheel_2" value="0.0" />
         <joint name="hip_yaw_3" value="0.0"/>
         <joint name="hip_pitch_3" value="1.0"/>
         <joint name="knee_pitch_3" value="1.0"/>
         <joint name="ankle_yaw_3" value="-0.78"/>
+        <joint name="ankle_pitch_3" value="0.0"/>
+        <joint name="j_wheel_3" value="0.0" />
         <joint name="hip_yaw_4" value="0.0"/>
         <joint name="hip_pitch_4" value="-1.0"/>
         <joint name="knee_pitch_4" value="-1.0"/>
         <joint name="ankle_yaw_4" value="0.78"/>
+        <joint name="ankle_pitch_4" value="0.0"/>
+        <joint name="j_wheel_4" value="0.0" />
+        <joint name="torso_yaw" value="0.0"/>
+        <joint name="neck_pitch" value="0.45"/>
     </group_state>
     <!--<group_state name="home" group="chains">

Commit message: Major step towards CENTAURO integration

File: robots/centauro_robot_description/config/centauro_srdf.xacro (robot description, xacro)
@@ -40,6 +40,6 @@
         <joint name="ankle_pitch_4"/>
         <joint name="j_wheel_4" />
-        <joint name="torso_yaw"/>
-        <joint name="neck_pitch" />
+        <!-- <joint name="torso_yaw"/>
+        <joint name="neck_pitch" /> -->
    </group>
    <group name="velodyne">
@@ -145,6 +145,6 @@
         <joint name="ankle_pitch_4" value="0.0"/>
         <joint name="j_wheel_4" value="0.0" />
-        <joint name="torso_yaw" value="0.0"/>
-        <joint name="neck_pitch" value="0.45"/>
+        <!-- <joint name="torso_yaw" value="0.0"/>
+        <joint name="neck_pitch" value="0.45"/> -->
     </group_state>
     <!--<group_state name="home" group="chains">

Commit message: Added Centauro URDF functionality with chosing joints, retrieving homing joints states, joint limits and more.

File: robots/centauro_robot_description/config/centauro_srdf.xacro (robot description, xacro)
@@ -108,5 +108,5 @@
    <group_state name="home" group="chains">
         <joint name="j_arm1_1" value="0.5"/>
-        <joint name="j_arm1_2" value="0.03"/>
+        <joint name="j_arm1_2" value="0.4"/>
         <joint name="j_arm1_3" value="-0.3"/>
         <joint name="j_arm1_4" value="-2.2"/>
@@ -115,5 +115,5 @@
         <joint name="j_arm1_7" value="0.0"/>
         <joint name="j_arm2_1" value="0.5"/>
-        <joint name="j_arm2_2" value="-0.03"/>
+        <joint name="j_arm2_2" value="-0.4"/>
         <joint name="j_arm2_3" value="0.3"/>
         <joint name="j_arm2_4" value="-2.2"/>
@@ -182,5 +182,5 @@
     </group_state>-->
     <group_state name="home_ank_yaw_0" group="chains">
-        <joint name="torso_yaw" value="0.0"/>
+        <!-- <joint name="torso_yaw" value="0.0"/> -->
         <joint name="j_arm1_1" value="0.0"/>
         <joint name="j_arm1_2" value="-0.3"/>
@@ -201,19 +201,27 @@
         <joint name="knee_pitch_1" value="0.8"/>
         <joint name="ankle_yaw_1" value="0.0"/>
+        <joint name="ankle_pitch_1" value="0.0"/>
+        <joint name="j_wheel_1" value="0.0" />
         <joint name="hip_yaw_2" value="-1.5"/>
         <joint name="hip_pitch_2" value="-0.8"/>
         <joint name="knee_pitch_2" value="-0.8"/>
         <joint name="ankle_yaw_2" value="0.0"/>
+        <joint name="ankle_pitch_2" value="0.0"/>
+        <joint name="j_wheel_2" value="0.0" />
         <joint name="hip_yaw_3" value="-1.5"/>
         <joint name="hip_pitch_3" value="-0.8"/>
         <joint name="knee_pitch_3" value="-0.8"/>
         <joint name="ankle_yaw_3" value="0.0"/>
+        <joint name="ankle_pitch_3" value="0.0"/>
+        <joint name="j_wheel_3" value="0.0" />
         <joint name="hip_yaw_4" value="1.5"/>
         <joint name="hip_pitch_4" value="0.8"/>
         <joint name="knee_pitch_4" value="0.8"/>
         <joint name="ankle_yaw_4" value="0.0"/>
+        <joint name="ankle_pitch_4" value="0.0"/>
+        <joint name="j_wheel_4" value="0.0" />
     </group_state>
     <group_state name="Zero_Pose" group="chains">
-        <joint name="torso_yaw" value="0.0"/>
+        <!-- <joint name="torso_yaw" value="0.0"/> -->
         <joint name="j_arm1_1" value="1.0"/>
         <joint name="j_arm1_2" value="-1.0"/>
@@ -233,24 +241,28 @@
         <joint name="hip_pitch_1" value="0.0"/>
         <joint name="knee_pitch_1" value="0.0"/>
+        <joint name="ankle_yaw_1" value="0.0"/>
         <joint name="ankle_pitch_1" value="0.0"/>
-        <joint name="ankle_yaw_1" value="0.0"/>
+        <joint name="j_wheel_1" value="0.0" />
         <joint name="hip_yaw_2" value="0.0"/>
         <joint name="hip_pitch_2" value="0.0"/>
         <joint name="knee_pitch_2" value="0.0"/>
+        <joint name="ankle_yaw_2" value="0.0"/>
         <joint name="ankle_pitch_2" value="0.0"/>
-        <joint name="ankle_yaw_2" value="0.0"/>
+        <joint name="j_wheel_2" value="0.0" />
         <joint name="hip_yaw_3" value="0.0"/>
         <joint name="hip_pitch_3" value="0.0"/>
         <joint name="knee_pitch_3" value="0.0"/>
+        <joint name="ankle_yaw_3" value="0.0"/>
         <joint name="ankle_pitch_3" value="0.0"/>
-        <joint name="ankle_yaw_3" value="0.0"/>
+        <joint name="j_wheel_3" value="0.0" />
         <joint name="hip_yaw_4" value="0.0"/>
         <joint name="hip_pitch_4" value="0.0"/>
         <joint name="knee_pitch_4" value="0.0"/>
+        <joint name="ankle_yaw_4" value="0.0"/>
         <joint name="ankle_pitch_4" value="0.0"/>
-        <joint name="ankle_yaw_4" value="0.0"/>
+        <joint name="j_wheel_4" value="0.0" />
     </group_state>
     <group_state name="Navvab_Parking_1" group="chains">
-        <joint name="torso_yaw" value="0.0"/>
+        <!-- <joint name="torso_yaw" value="0.0"/> -->
         <joint name="j_arm1_1" value="1.57"/>
         <joint name="j_arm1_2" value="0.1"/>
@@ -270,24 +282,28 @@
         <joint name="hip_pitch_1" value="-1.57"/>
         <joint name="knee_pitch_1" value="2.44"/>
+        <joint name="ankle_yaw_1" value="0.0"/>
         <joint name="ankle_pitch_1" value="2.44"/>
-        <joint name="ankle_yaw_1" value="0.0"/>
+        <joint name="j_wheel_1" value="0.0" />
         <joint name="hip_yaw_2" value="0.0"/>
         <joint name="hip_pitch_2" value="1.57"/>
         <joint name="knee_pitch_2" value="-2.44"/>
+        <joint name="ankle_yaw_2" value="0.0"/>
         <joint name="ankle_pitch_2" value="-2.44"/>
-        <joint name="ankle_yaw_2" value="0.0"/>
+        <joint name="j_wheel_2" value="0.0" />
         <joint name="hip_yaw_3" value="0.0"/>
         <joint name="hip_pitch_3" value="1.57"/>
         <joint name="knee_pitch_3" value="-2.44"/>
+        <joint name="ankle_yaw_3" value="0.0"/>
         <joint name="ankle_pitch_3" value="-2.44"/>
-        <joint name="ankle_yaw_3" value="0.0"/>
+        <joint name="j_wheel_3" value="0.0" />
         <joint name="hip_yaw_4" value="0.0"/>
         <joint name="hip_pitch_4" value="-1.57"/>
         <joint name="knee_pitch_4" value="2.44"/>
+        <joint name="ankle_yaw_4" value="0.0"/>
         <joint name="ankle_pitch_4" value="2.44"/>
-        <joint name="ankle_yaw_4" value="0.0"/>
+        <joint name="j_wheel_4" value="0.0" />
     </group_state>
     <group_state name="Navvab_Parking_2" group="chains">
-        <joint name="torso_yaw" value="0.0"/>
+        <!-- <joint name="torso_yaw" value="0.0"/> -->
         <joint name="j_arm1_1" value="1.57"/>
         <joint name="j_arm1_2" value="0.1"/>
@@ -307,24 +323,28 @@
         <joint name="hip_pitch_1" value="-1.83"/>
         <joint name="knee_pitch_1" value="-2.44"/>
+        <joint name="ankle_yaw_1" value="0.0"/>
         <joint name="ankle_pitch_1" value="0.7"/>
-        <joint name="ankle_yaw_1" value="0.0"/>
+        <joint name="j_wheel_1" value="0.0" />
         <joint name="hip_yaw_2" value="0.0"/>
         <joint name="hip_pitch_2" value="1.83"/>
         <joint name="knee_pitch_2" value="2.44"/>
+        <joint name="ankle_yaw_2" value="0.0"/>
         <joint name="ankle_pitch_2" value="-0.7"/>
-        <joint name="ankle_yaw_2" value="0.0"/>
+        <joint name="j_wheel_2" value="0.0" />
         <joint name="hip_yaw_3" value="0.0"/>
         <joint name="hip_pitch_3" value="1.83"/>
         <joint name="knee_pitch_3" value="2.44"/>
+        <joint name="ankle_yaw_3" value="0.0"/>
         <joint name="ankle_pitch_3" value="-0.7"/>
-        <joint name="ankle_yaw_3" value="0.0"/>
+        <joint name="j_wheel_3" value="0.0" />
         <joint name="hip_yaw_4" value="0.0"/>
         <joint name="hip_pitch_4" value="-1.83"/>
         <joint name="knee_pitch_4" value="-2.44"/>
+        <joint name="ankle_yaw_4" value="0.0"/>
         <joint name="ankle_pitch_4" value="0.7"/>
-        <joint name="ankle_yaw_4" value="0.0"/>
+        <joint name="j_wheel_4" value="0.0" />
     </group_state>
     <group_state name="Navvab_Parking_3" group="chains">
-        <joint name="torso_yaw" value="0.0"/>
+        <!-- <joint name="torso_yaw" value="0.0"/> -->
         <joint name="j_arm1_1" value="1.57"/>
         <joint name="j_arm1_2" value="0.1"/>
@@ -344,24 +364,28 @@
         <joint name="hip_pitch_1" value="-1.83"/>
         <joint name="knee_pitch_1" value="-2.44"/>
+        <joint name="ankle_yaw_1" value="0.0"/>
         <joint name="ankle_pitch_1" value="-2.44"/>
-        <joint name="ankle_yaw_1" value="0.0"/>
+        <joint name="j_wheel_1" value="0.0" />
         <joint name="hip_yaw_2" value="0.0"/>
         <joint name="hip_pitch_2" value="1.83"/>
         <joint name="knee_pitch_2" value="2.44"/>
+        <joint name="ankle_yaw_2" value="0.0"/>
         <joint name="ankle_pitch_2" value="2.44"/>
-        <joint name="ankle_yaw_2" value="0.0"/>
+        <joint name="j_wheel_2" value="0.0" />
         <joint name="hip_yaw_3" value="0.0"/>
         <joint name="hip_pitch_3" value="1.83"/>
         <joint name="knee_pitch_3" value="2.44"/>
+        <joint name="ankle_yaw_3" value="0.0"/>
         <joint name="ankle_pitch_3" value="2.44"/>
-        <joint name="ankle_yaw_3" value="0.0"/>
+        <joint name="j_wheel_3" value="0.0" />
         <joint name="hip_yaw_4" value="0.0"/>
         <joint name="hip_pitch_4" value="-1.83"/>
         <joint name="knee_pitch_4" value="-2.44"/>
+        <joint name="ankle_yaw_4" value="0.0"/>
         <joint name="ankle_pitch_4" value="-2.44"/>
-        <joint name="ankle_yaw_4" value="0.0"/>
+        <joint name="j_wheel_4" value="0.0" />
     </group_state>
     <group_state name="Navvab_Parking_4" group="chains">
-        <joint name="torso_yaw" value="0.0"/>
+        <!-- <joint name="torso_yaw" value="0.0"/> -->
         <joint name="j_arm1_1" value="1.57"/>
         <joint name="j_arm1_2" value="0.1"/>
@@ -381,21 +405,25 @@
         <joint name="hip_pitch_1" value="0.52"/>
         <joint name="knee_pitch_1" value="2.44"/>
+        <joint name="ankle_yaw_1" value="0.0"/>
         <joint name="ankle_pitch_1" value="2.44"/>
-        <joint name="ankle_yaw_1" value="0.0"/>
+        <joint name="j_wheel_1" value="0.0" />
         <joint name="hip_yaw_2" value="0.0"/>
         <joint name="hip_pitch_2" value="-0.52"/>
         <joint name="knee_pitch_2" value="-2.44"/>
+        <joint name="ankle_yaw_2" value="0.0"/>
         <joint name="ankle_pitch_2" value="-2.44"/>
-        <joint name="ankle_yaw_2" value="0.0"/>
+        <joint name="j_wheel_2" value="0.0" />
         <joint name="hip_yaw_3" value="0.0"/>
         <joint name="hip_pitch_3" value="-0.52"/>
         <joint name="knee_pitch_3" value="-2.44"/>
+        <joint name="ankle_yaw_3" value="0.0"/>
         <joint name="ankle_pitch_3" value="-2.44"/>
-        <joint name="ankle_yaw_3" value="0.0"/>
+        <joint name="j_wheel_3" value="0.0" />
         <joint name="hip_yaw_4" value="0.0"/>
         <joint name="hip_pitch_4" value="0.52"/>
         <joint name="knee_pitch_4" value="2.44"/>
+        <joint name="ankle_yaw_4" value="0.0"/>
         <joint name="ankle_pitch_4" value="2.44"/>
-        <joint name="ankle_yaw_4" value="0.0"/>
+        <joint name="j_wheel_4" value="0.0" />
     </group_state>
 </robot>

File: robots/centauro_robot_description/config/joint_limits.xacro (robot description, xacro)
@@ -50,3 +50,9 @@
 <xacro:property name="motor_B_effort" value="147"/>
 <xacro:property name="motor_C_effort" value="35"/>
+<motor name="hip_yaw" value="motor_A" />
+<motor name="hip_pitch" value="motor_A" />
+<motor name="knee_pitch" value="motor_A" />
+<motor name="ankle_yaw" value="motor_C" />
+<motor name="ankle_pitch" value="motor_B" />
+<motor name="j_wheel" value="motor_C" />
 </robot>

Commit message: Playing with different hitting directions --> changing cost functions Also removed some files and changed up some of the base functions

File: robots/centauro_robot_description/config/centauro_srdf.xacro (robot description, xacro)
@@ -107,4 +107,47 @@
    </group>
    <group_state name="home" group="chains">
+        <joint name="j_arm1_1" value="0.520149"/>
+        <joint name="j_arm1_2" value="0.320865"/>
+        <joint name="j_arm1_3" value="0.274669"/>
+        <joint name="j_arm1_4" value="-2.23604"/>
+        <joint name="j_arm1_5" value="0.0500815"/>
+        <joint name="j_arm1_6" value="-0.781461"/>
+        <joint name="j_arm1_7" value="-0.0567608"/>
+        <joint name="j_arm2_1" value="0.520149"/>
+        <joint name="j_arm2_2" value="-0.320865"/>
+        <joint name="j_arm2_3" value="-0.274669"/>
+        <joint name="j_arm2_4" value="-2.23604"/>
+        <joint name="j_arm2_5" value="-0.0500815"/>
+        <joint name="j_arm2_6" value="-0.781461"/>
+        <joint name="j_arm2_7" value="0.0567608"/>
+        <joint name="hip_yaw_1" value="-0.746874"/>
+        <joint name="hip_pitch_1" value="-1.25409"/>
+        <joint name="knee_pitch_1" value="-1.55576"/>
+        <joint name="ankle_yaw_1" value="0.746874"/>
+        <joint name="ankle_pitch_1" value="-0.301666"/>
+        <joint name="j_wheel_1" value="0.0" />
+        <joint name="hip_yaw_2" value="0.746874"/>
+        <joint name="hip_pitch_2" value="1.25409"/>
+        <joint name="knee_pitch_2" value="1.55576"/>
+        <joint name="ankle_yaw_2" value="-0.746874"/>
+        <joint name="ankle_pitch_2" value="0.301666"/>
+        <joint name="j_wheel_2" value="0.0" />
+        <joint name="hip_yaw_3" value="0.746874"/>
+        <joint name="hip_pitch_3" value="1.25409"/>
+        <joint name="knee_pitch_3" value="1.55576"/>
+        <joint name="ankle_yaw_3" value="-0.746874"/>
+        <joint name="ankle_pitch_3" value="0.301667"/>
+        <joint name="j_wheel_3" value="0.0" />
+        <joint name="hip_yaw_4" value="-0.746874"/>
+        <joint name="hip_pitch_4" value="-1.25409"/>
+        <joint name="knee_pitch_4" value="-1.55576"/>
+        <joint name="ankle_yaw_4" value="0.746874"/>
+        <joint name="ankle_pitch_4" value="-0.301667"/>
+        <joint name="j_wheel_4" value="0.0" /> -->
+        <!-- <joint name="torso_yaw" value="3.56617e-13"/>
+        <joint name="neck_yaw" value="1.22719e-16"/>
+        <joint name="neck_pitch" value="0.45"/> -->
+    </group_state>
+    <group_state name="home_old" group="chains">
         <joint name="j_arm1_1" value="0.5"/>
         <joint name="j_arm1_2" value="0.4"/>
@@ -148,6 +191,6 @@
         <joint name="neck_pitch" value="0.45"/> -->
     </group_state>
-    <!--<group_state name="home" group="chains">
-        <joint name="torso_yaw" value="0.0"/>
+    <group_state name="home_ank_yaw_0" group="chains">
+        <!-- <joint name="torso_yaw" value="0.0"/> -->
         <joint name="j_arm1_1" value="0.0"/>
         <joint name="j_arm1_2" value="-0.3"/>
@@ -167,37 +210,4 @@
         <joint name="hip_pitch_1" value="0.8"/>
         <joint name="knee_pitch_1" value="0.8"/>
-        <joint name="ankle_yaw_1" value="1.5"/>
-        <joint name="hip_yaw_2" value="-1.5"/>
-        <joint name="hip_pitch_2" value="-0.8"/>
-        <joint name="knee_pitch_2" value="-0.8"/>
-        <joint name="ankle_yaw_2" value="-1.5"/>
-        <joint name="hip_yaw_3" value="-1.5"/>
-        <joint name="hip_pitch_3" value="-0.8"/>
-        <joint name="knee_pitch_3" value="-0.8"/>
-        <joint name="ankle_yaw_3" value="-1.5"/>
-        <joint name="hip_yaw_4" value="1.5"/>
-        <joint name="hip_pitch_4" value="0.8"/>
-        <joint name="knee_pitch_4" value="0.8"/>
-        <joint name="ankle_yaw_4" value="1.5"/>
-    </group_state>-->
-    <group_state name="home_ank_yaw_0" group="chains">
-        <!-- <joint name="torso_yaw" value="0.0"/> -->
-        <joint name="j_arm1_1" value="0.0"/>
-        <joint name="j_arm1_2" value="-0.3"/>
-        <joint name="j_arm1_3" value="-0.8"/>
-        <joint name="j_arm1_4" value="-0.8"/>
-        <joint name="j_arm1_5" value="-0.0"/>
-        <joint name="j_arm1_6" value="-0.8"/>
-        <joint name="j_arm1_7" value="0.0"/>
-        <joint name="j_arm2_1" value="0.0"/>
-        <joint name="j_arm2_2" value="0.3"/>
-        <joint name="j_arm2_3" value="0.8"/>
-        <joint name="j_arm2_4" value="0.8"/>
-        <joint name="j_arm2_5" value="0.0"/>
-        <joint name="j_arm2_6" value="0.8"/>
-        <joint name="j_arm2_7" value="0.0"/>
-        <joint name="hip_yaw_1" value="1.5"/>
-        <joint name="hip_pitch_1" value="0.8"/>
-        <joint name="knee_pitch_1" value="0.8"/>
         <joint name="ankle_yaw_1" value="0.0"/>
         <joint name="ankle_pitch_1" value="0.0"/>
