Commit message: Major update: Fixed some issues in optization. Now running correct optimization. 7DoF system added with Torso. Ready to test a horizontal Punch motion.

File: robots/centauro_robot_description/config/centauro_srdf.xacro (robot description, xacro)
@@ -2,4 +2,5 @@
 <robot name="centauro">
    <group name="joint_names">
+        <joint name="torso_yaw"/>
         <joint name="j_arm1_1" />
         <joint name="j_arm1_2" />
@@ -40,6 +41,5 @@
         <joint name="ankle_pitch_4"/>
         <joint name="j_wheel_4" />
-        <!-- <joint name="torso_yaw"/>
-        <joint name="neck_pitch" /> -->
+                <!-- <joint name="neck_pitch" /> -->
    </group>
    <group name="velodyne">
@@ -107,4 +107,5 @@
    </group>
    <group_state name="home" group="chains">
+        <joint name="torso_yaw" value="3.56617e-13"/>
         <joint name="j_arm1_1" value="0.520149"/>
         <joint name="j_arm1_2" value="0.320865"/>
@@ -145,9 +146,9 @@
         <joint name="ankle_pitch_4" value="-0.301667"/>
         <joint name="j_wheel_4" value="0.0" /> -->
-        <!-- <joint name="torso_yaw" value="3.56617e-13"/>
-        <joint name="neck_yaw" value="1.22719e-16"/>
+        <!-- <joint name="neck_yaw" value="1.22719e-16"/>
         <joint name="neck_pitch" value="0.45"/> -->
     </group_state>
     <group_state name="home_old" group="chains">
+        <joint name="torso_yaw" value="0.0"/>
         <joint name="j_arm1_1" value="0.5"/>
         <joint name="j_arm1_2" value="0.4"/>
@@ -188,9 +189,7 @@
         <joint name="ankle_pitch_4" value="0.0"/>
         <joint name="j_wheel_4" value="0.0" />
-        <!-- <joint name="torso_yaw" value="0.0"/>
-        <joint name="neck_pitch" value="0.45"/> -->
+        <!-- <joint name="neck_pitch" value="0.45"/> -->
     </group_state>
     <group_state name="home_ank_yaw_0" group="chains">
-        <!-- <joint name="torso_yaw" value="0.0"/> -->
         <joint name="j_arm1_1" value="0.0"/>
         <joint name="j_arm1_2" value="-0.3"/>
@@ -231,4 +230,5 @@
         <joint name="ankle_pitch_4" value="0.0"/>
         <joint name="j_wheel_4" value="0.0" />
+        <joint name="torso_yaw" value="0.0"/>
     </group_state>
     <group_state name="Zero_Pose" group="chains">

File: robots/centauro_robot_description/config/joint_limits.xacro (robot description, xacro)
@@ -14,6 +14,8 @@
 <xacro:property name="ankle_yaw_lower" value="${[-2.5626, -2.5546, -2.5606, -2.6046]}"/>
 <xacro:property name="ankle_yaw_upper" value="${[ 2.5384,  2.5484,  2.5454,  2.5514]}"/>
-<xacro:property name="torso_yaw_lower" value="-2.618"/>
-<xacro:property name="torso_yaw_upper" value="2.618"/>
+<!-- <xacro:property name="torso_yaw_lower" value="-2.618"/>
+<xacro:property name="torso_yaw_upper" value="2.618"/> -->
+<xacro:property name="torso_yaw_lower" value="${[-1.0]}"/>
+<xacro:property name="torso_yaw_upper" value="${[1.0]}"/>
 <xacro:property name="j_arm_1_lower" value="${[-3.312, -3.3458]}"/>
 <xacro:property name="j_arm_2_lower" value="${[ 0.020, -3.4258]}"/>
@@ -62,7 +64,9 @@
 <xacro:property name="motor_B_velocity" value="8.1"/>
 <xacro:property name="motor_C_velocity" value="20.0"/>
+<xacro:property name="motor_D_velocity" value="5.7"/>
 <xacro:property name="motor_A_effort" value="304"/>
 <xacro:property name="motor_B_effort" value="147"/>
 <xacro:property name="motor_C_effort" value="35"/>
+<xacro:property name="motor_D_effort" value="147"/>
 <motor name="hip_yaw" value="motor_A" />
 <motor name="hip_pitch" value="motor_A" />
@@ -71,3 +75,4 @@
 <motor name="ankle_pitch" value="motor_B" />
 <motor name="j_wheel" value="motor_C" />
+<motor name="torso_yaw" value="motor_D" />
 </robot>
